Commit message: Separate robot materials into xacro module

File: my_robot/urdf/robot.urdf.xacro (robot description, xacro)
@@ -1,14 +1,6 @@
 <?xml version="1.0"?>
 <robot xmlns:xacro="http://www.ros.org/wiki/xacro" name="warehouse_bot">
+  <xacro:include filename="$(find my_robot)/urdf/materials.xacro"/>
   <!-- ================= MATERIALS ================= -->
-  <material name="body_blue">
-    <color rgba="0.05 0.25 0.8 1"/>
-  </material>
-  <material name="dark_gray">
-    <color rgba="0.15 0.15 0.15 1"/>
-  </material>
-  <material name="silver">
-    <color rgba="0.7 0.7 0.7 1"/>
-  </material>
   <!-- ================= MAIN BODY ================= -->
   <link name="base_link">

Commit message: Move chassis into separate xacro module

File: my_robot/urdf/robot.urdf.xacro (robot description, xacro)
@@ -2,53 +2,8 @@
 <robot xmlns:xacro="http://www.ros.org/wiki/xacro" name="warehouse_bot">
   <xacro:include filename="$(find my_robot)/urdf/materials.xacro"/>
+  <xacro:include filename="$(find my_robot)/urdf/chassis.xacro"/>
   <!-- ================= MATERIALS ================= -->
   <!-- ================= MAIN BODY ================= -->
-  <link name="base_link">
-    <visual>
-      <origin xyz="0 0 0.18"/>
-      <geometry>
-        <box size="0.65 0.45 0.25"/>
-      </geometry>
-      <material name="body_blue"/>
-    </visual>
-    <collision>
-      <origin xyz="0 0 0.18"/>
-      <geometry>
-        <box size="0.65 0.45 0.25"/>
-      </geometry>
-    </collision>
-    <inertial>
-      <origin xyz="0 0 0.18"/>
-      <mass value="6"/>
-      <inertia
-        ixx="0.2"
-        ixy="0"
-        ixz="0"
-        iyy="0.2"
-        iyz="0"
-        izz="0.2"/>
-    </inertial>
-  </link>
   <!-- ================= TOP SENSOR PLATFORM ================= -->
-  <link name="top_plate">
-    <visual>
-      <origin xyz="0 0 0.34"/>
-      <geometry>
-        <box size="0.35 0.30 0.04"/>
-      </geometry>
-      <material name="silver"/>
-    </visual>
-    <collision>
-      <origin xyz="0 0 0.34"/>
-      <geometry>
-        <box size="0.35 0.30 0.04"/>
-      </geometry>
-    </collision>
-  </link>
-  <joint name="top_plate_joint" type="fixed">
-    <parent link="base_link"/>
-    <child link="top_plate"/>
-    <origin xyz="0 0 0"/>
-  </joint>
   <!-- ================= LEFT WHEEL ================= -->
   <link name="left_wheel">

Commit message: Separate wheels and caster into xacro module

File: my_robot/urdf/robot.urdf.xacro (robot description, xacro)
@@ -3,92 +3,11 @@
   <xacro:include filename="$(find my_robot)/urdf/materials.xacro"/>
   <xacro:include filename="$(find my_robot)/urdf/chassis.xacro"/>
+  <xacro:include filename="$(find my_robot)/urdf/wheels.xacro"/>
   <!-- ================= MATERIALS ================= -->
   <!-- ================= MAIN BODY ================= -->
   <!-- ================= TOP SENSOR PLATFORM ================= -->
   <!-- ================= LEFT WHEEL ================= -->
-  <link name="left_wheel">
-    <visual>
-      <origin rpy="1.5708 0 0"/>
-      <geometry>
-        <cylinder radius="0.11" length="0.06"/>
-      </geometry>
-      <material name="dark_gray"/>
-    </visual>
-    <collision>
-      <origin rpy="1.5708 0 0"/>
-      <geometry>
-        <cylinder radius="0.11" length="0.06"/>
-      </geometry>
-    </collision>
-    <inertial>
-      <mass value="1"/>
-      <inertia
-        ixx="0.01"
-        ixy="0"
-        ixz="0"
-        iyy="0.01"
-        iyz="0"
-        izz="0.01"/>
-    </inertial>
-  </link>
   <!-- ================= RIGHT WHEEL ================= -->
-  <link name="right_wheel">
-    <visual>
-      <origin rpy="1.5708 0 0"/>
-      <geometry>
-        <cylinder radius="0.11" length="0.06"/>
-      </geometry>
-      <material name="dark_gray"/>
-    </visual>
-    <collision>
-      <origin rpy="1.5708 0 0"/>
-      <geometry>
-        <cylinder radius="0.11" length="0.06"/>
-      </geometry>
-    </collision>
-    <inertial>
-      <mass value="1"/>
-      <inertia
-        ixx="0.01"
-        ixy="0"
-        ixz="0"
-        iyy="0.01"
-        iyz="0"
-        izz="0.01"/>
-    </inertial>
-  </link>
   <!-- ================= WHEEL JOINTS ================= -->
-  <joint name="left_wheel_joint" type="continuous">
-    <parent link="base_link"/>
-    <child link="left_wheel"/>
-    <origin xyz="0 0.27 0.11"/>
-    <axis xyz="0 1 0"/>
-  </joint>
-  <joint name="right_wheel_joint" type="continuous">
-    <parent link="base_link"/>
-    <child link="right_wheel"/>
-    <origin xyz="0 -0.27 0.11"/>
-    <axis xyz="0 1 0"/>
-  </joint>
-  <!-- ================= REAR CASTER ================= -->
-  <link name="caster_wheel">
-    <visual>
-      <geometry>
-        <sphere radius="0.05"/>
-      </geometry>
-      <origin xyz="-0.25 0 0.05"/>
-      <material name="dark_gray"/>
-    </visual>
-    <collision>
-      <geometry>
-        <sphere radius="0.05"/>
-      </geometry>
-      <origin xyz="-0.25 0 0.05"/>
-    </collision>
-  </link>
-  <joint name="caster_joint" type="fixed">
-    <parent link="base_link"/>
-    <child link="caster_wheel"/>
-    <origin xyz="0 0 0"/>
-  </joint>
+  <!-- ================= REAR CASTER =========================-->
 </robot>

Commit message: Release v1.0.0 of Autonomous Warehouse Robot

File: my_robot/urdf/robot.urdf.xacro (robot description, xacro)
@@ -4,4 +4,5 @@
   <xacro:include filename="$(find my_robot)/urdf/chassis.xacro"/>
   <xacro:include filename="$(find my_robot)/urdf/wheels.xacro"/>
+  <xacro:include filename="$(find my_robot)/urdf/gazebo.xacro"/>
   <!-- ================= MATERIALS ================= -->
   <!-- ================= MAIN BODY ================= -->

File: my_robot/urdf/warehouse_bot.urdf (robot description, URDF)
Before this commit: robot warehouse_bot, 5 links, 4 joints
Links:
- added link base_footprint
- added link imu_link, mass 0.05; collision box size=0.06 0.04 0.02; visual box size=0.06 0.04 0.02
- added link lidar_link, mass 0.25; collision cylinder length=0.06 radius=0.07; visual cylinder length=0.06 radius=0.07
- link base_link: mass 6 -> 6.0
- link caster_wheel: mass None -> 0.2
- link left_wheel: mass 1 -> 1.0
- link right_wheel: mass 1 -> 1.0
- link top_plate: mass None -> 0.4
Joints:
- added joint base_footprint_joint: type fixed, parent base_footprint, child base_link, origin xyz=0 0 0
- added joint imu_joint: type fixed, parent base_link, child imu_link, origin xyz=0 0 0.22
- added joint lidar_joint: type fixed, parent top_plate, child lidar_link, origin xyz=0 0 0.07
- joint caster_joint: origin xyz=0 0 0 -> xyz=-0.25 0 0.05
- joint top_plate_joint: origin xyz=0 0 0 -> xyz=0 0 0.34
